Commit message: Updates for ethercat Checking

File: tocabi_description/robots/dyros_tocabi.urdf (robot description, URDF)
Before this commit: robot dyros_tocabi_description, 36 links, 35 joints
Links:
- link Head_Link: mass 0.006332 -> 2.006332

Commit message: update urdf/xml inertial information

File: tocabi_description/robots/dyros_tocabi.urdf (robot description, URDF)
Before this commit: robot dyros_tocabi_description, 36 links, 35 joints
Links:
- link Head_Link: mass 2.006332 -> 1.417
