Commit message: update head stl, display

File: tocabi_description/robots/dyros_tocabi_0714.urdf (robot description, URDF)
Before this commit: robot dyros_tocabi_description, 36 links, 35 joints
Links:
- link Head_Link: geometry collision cylinder length=0.043 radius=0.07; visual mesh filename=package://tocabi_description/meshes/head_v1.stl scale=0.001 0.001 0.001
- link L_Wrist2_Link: geometry collision box size=0.06 0.06 0.02; visual box size=0.03 0.005 0.05
- link R_Wrist2_Link: geometry collision box size=0.06 0.06 0.02; visual box size=0.03 0.005 0.05
